File: PWM-TRANSISTOR-PCB/PWM-TRANSISTOR-PCB.kicad_pcb (KiCad board)
At the start: 2 copper layers, 26.4 x 23.9 mm, 13 parts, among them J1 MOTOR_CON, J2 Screw_Terminal_01x02, J3 PWM_IN, J4 VCC_CON, Q1 2N2222A

Commit message: Añadidos las README así como GERBERS y RENDERs
Parts:
- removed G***: LOGO, Logo:Logo_DC
Other:
- board text added: "Github: AugustoS97"
- board text removed: "digitalcodesign.com"
